File: schematics/gc-1000-gps.brd (EAGLE design)
At the start: 161.3 x 130.1 mm, 17 parts, among them T1 2N3904

Commit message: Import v0.2
Parts:
- added SPKR: 22-23-2021, con-molex:22-23-2021
- C1: value (none) -> 0.1µF
- C2: value (none) -> 10µF
- J1: value (none) -> 12v
- moved C2 3.81 mm to (21.6, 11.4)
- moved C1 1.80 mm to (17.8, 26.7)
- renumbered H1 to J2, T1 to Q1, U$3 to U1
Connections:
- net N$21 renamed DISP6
- net N$23 renamed DISP5
- net N$24 renamed DISP4
- net N$25 renamed DISP3
- net N$26 renamed DISP2
- net N$27 renamed DISP1
- net N$28 renamed DISP0
- net N$34 renamed DISP7
- net N$35 renamed DISP8
- net N$36 renamed DISP9
- net N$37 renamed DISP10
- net N$38 renamed DISP11
- net N$39 renamed DISP12
- net N$40 renamed 7SEG2
- net N$41 renamed 7SEG1
- net N$42 renamed 7SEG0
- removed net N$29: U$6.P$11, U$7.P$11
- new net CLK: B1.12, U$6.P$11, U$7.P$11
- new net DATPIN: B1.11, U$6.P$14
- new net LATCH: B1.8, U$6.P$12, U$7.P$12
- new net N$21: B1.4, SPKR.1
- net GND: now also SPKR.2
Routing:
- net CLK: track 0.00 -> 234.1 mm, vias 0 -> 4
- net LATCH: track 0.00 -> 220.6 mm, vias 0 -> 1
- net DATPIN: track 0.00 -> 219.8 mm, vias 0 -> 2
- net B$2: track 115.9 -> 259.8 mm, vias 0 -> 4
- net N$22: track 114.3 -> 180.4 mm, vias 3 -> 0
- net N$21: track 0.00 -> 65.0 mm, vias 0 -> 1
- net N$5: track 157.0 -> 216.5 mm, vias 0 -> 3
- net N$51: track 151.5 -> 184.8 mm, vias 0 -> 1
- net N$61: track 107.9 -> 140.5 mm, vias 1 -> 4
- net N$10: track 157.3 -> 128.5 mm, vias 0 -> 1
- net DISP8: track 63.1 -> 91.3 mm
- net N$44: track 33.5 -> 59.7 mm, vias 0 -> 3
- net N$29: track 26.0 -> 0.00 mm
- net N$11: track 128.4 -> 152.4 mm, vias 1 -> 2
- net N$45: track 34.3 -> 56.9 mm
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Other:
- board text added: "13"
- board text added: "2"
- board text added: "2N3904"
- board text added: "ON"
- board text added: "gc-1000-gps www.ac1ja.com v0.2"
- board text removed: "gc-1000-gps www.ac1ja.com v0.1-lw-132-g480f"
