File: hardware/gc-1000-gps/gc-1000-gps.kicad_sch (KiCad schematic)
At the start: 18 parts, among them J1 12v, J2 MA07-2, Q1 2N3904, SW1 SW_DIP-8, SW2 SW_DIP-8, U1 OKI-78SR, X1 F25HPS

Commit message: Add BOM generator
Parts:
- B1: LINK (none) -> https://store.arduino.cc/products/arduino-mega-2560-rev3
- U$1: LINK (none) -> https://www.adafruit.com/product/746
- U$4: LINK (none) -> https://www.adafruit.com/product/3013
Changed lines of the file:
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@@
+      (effects (font (size 1.27 1.27)) hide)
+    )
+    (property "LINK" "https://store.arduino.cc/products/arduino-mega-2560-rev3" (at 79.375 97.79 0)
       (effects (font (size 1.27 1.27)) hide)
     )
@@
       (effects (font (size 1.27 1.27)) hide)
     )
+    (property "LINK" "https://www.adafruit.com/product/3013" (at 155.575 59.69 0)
+      (effects (font (size 1.27 1.27)) hide)
+    )
     (pin "P$1")
     (pin "P$2")
@@
       (effects (font (size 1.27 1.27)) hide)
     )
+    (property "LINK" "https://www.adafruit.com/product/746" (at 150.495 19.05 0)
+      (effects (font (size 1.27 1.27)) hide)
+    )
